File: hardware/wrist_board/_autosave-wrist_board.kicad_sch (KiCad schematic)
At the start: 5 parts, among them P1 USB_C_Plug_USB2.0, U1 MCP73831T-2ACI_OT

Commit message: Minor updates to charging circuit
Parts:
- added C2: 4.7uF, symbol Device:C_Small_US
- added D1: Charging LED, symbol Device:LED
- added J1: S2B-PH-K-S_LF__SN_, S2B-PH-K-S_LF__SN_:JST_S2B-PH-K-S_LF__SN_, symbol S2B-PH-K-S_LF__SN_:S2B-PH-K-S_LF__SN_
- added R3: 2k, symbol Device:R_Small
- added R4: 470, symbol Device:R_Small
- C1: value 22uF -> 10uF
Connections:
- net GND: now also C2.2
- net at U1.1 (STAT): now also R4.1
- net at U1.2 (VSS): now also R3.2
- net at U1.3 (VBAT): no longer names the net of U1.3 (VBAT)
- net at U1.3 (VBAT): now also C2.1
- net at U1.4 (VDD): now also D1.2 (A)
- net at U1.5 (PROG): now also R3.1
- new net: D1.1 (K), R4.2
Other:
- moved on the sheet: U1
