File: hardware/processing_board/_autosave-processing_board.kicad_sch (KiCad schematic)
At the start: 50 parts, among them J1 USB_C_Receptacle_USB2.0_14P, J2 USB_C_Receptacle_USB2.0_14P, J3 S2B-PH-K-S_LF__SN_, U1 BQ24075RGT, U2 NCP1117-3.3_SOT223, U3 TPS62821DLC, U4 TPS22917DBV, U5 NCP1117-1.8_SOT223, U6 FT2232HQ, Y1 Crystal

Commit message: Added FPGA bypass caps
Parts:
- added C18, C19, C20, C21, C22, C23, C24, C25, C28, C31: 0.1uF, symbol Device:C_Small_US
- added C26, C32, C33, C41, C42, C47, C48, C55, C56, C60, C61, C71, C72, C73: 47nF, symbol Device:C_Small_US
- added C27, C34, C35, C36, C37, C43, C44, C45, C46, C49, C50, C51, C52, C57, C62, C63, C66, C67, C74, C75: 470nF, symbol Device:C_Small_US
- added C29: 100nF, symbol Device:C_Small_US
- added C30: 0.1uF, Capacitor_SMD:C_0805_2012Metric, symbol Device:C_Small_US
- added C38, C39, C53, C54, C59, C64, C68, C69: 4.7uF, symbol Device:C_Small_US
- added C40, C70: 100uF, symbol Device:C_Small_US
- added C58, C65: 47uF, symbol Device:C_Small_US
- added C76: 10nF, symbol Device:C_Small_US
- added FB1, FB2: 600@100MHZ, symbol Device:FerriteBead_Small
- added IC1: XC7S25-2CSGA225I, BGA225C80P15X15_1300X1300X140, symbol XC7S25-2CSGA225I:XC7S25-2CSGA225I
- added J4: Micro_SD_Card_Det1, symbol Connector:Micro_SD_Card_Det1
- added R16, R17: 1k, symbol Device:R_Small
- added R21: 2.2k, symbol Device:R_Small
- added R22: 330, symbol Device:R_Small
- added R23: 4.7k, symbol Device:R_Small
- added R24: 10k, symbol Device:R_Small
- added R25, R26: 10k, Resistor_SMD:R_0805_2012Metric, symbol Device:R_Small
- added SW1: SW_Push, symbol Switch:SW_Push
- added SW2: BOOT_BTN, Button_Switch_SMD:SW_SPST_B3U-1000P, symbol Switch:SW_Push
- added SW3: RST_BTN, Button_Switch_SMD:SW_SPST_B3U-1000P, symbol Switch:SW_Push
- added U7: 93LCxxA, symbol Memory_EEPROM:93LCxxA
- added U8: W25Q32JVSS, Package_SO:SOIC-8_5.3x5.3mm_P1.27mm, symbol Memory_Flash:W25Q32JVSS
- added X1: ESP32-S3-WROOM-1-N16R8, ESP32-S3-WROOM-1-N16R8:ESP32S3WROOM1N8R2, symbol ESP32-S3-WROOM-1-N16R8:ESP32-S3-WROOM-1-N16R8
- added Y2: ECS-2520MV-xxx-xx, Oscillator:Oscillator_SMD_ECS_2520MV-xxx-xx-4Pin_2.5x2.0mm, symbol Oscillator:ECS-2520MV-xxx-xx
Connections:
- net +1V0: now also C55.1, C56.1, C57.1, C58.1, C59.1, C66.1, C67.1, C68.1, C69.1, C70.1, C71.1, C72.1, C73.1, C74.1, IC1.E10 (VCCINT_2), IC1.E8 (VCCINT_1), IC1.F7 (VCCINT_3), IC1.G10 (VCCINT_4), IC1.G6 (VCCBRAM_1), IC1.H7 (VCCINT_5), IC1.J10 (VCCINT_6), IC1.J6 (VCCBRAM_2), IC1.K7 (VCCINT_7), IC1.K9 (VCCINT_8)
- net +1V8: now also C60.1, C61.1, C62.1, C63.1, C64.1, C65.1, FB1.1, IC1.L6 (VCCAUX_1), IC1.L8 (VCCAUX_2)
- net +3V3: now also U6.19 (ADBUS3), C18.1, C28.1, C29.1, C30.1, C31.1, IC1.H5 (CFGBVS_0), J4.4 (VDD), R16.1, R22.1, R23.2, R24.1, R25.2, R26.2, U7.8 (VCC), U8.8 (VCC), X1.2 (3V3), Y2.1 (Tri-State), Y2.4 (VDD)
- net 3V3_FPGA: now also C26.1, C27.1, C32.1, C33.1, C34.1, C35.1, C36.1, C37.1, C38.1, C39.1, C40.1, C41.1, C42.1, C43.1, C44.1, C45.1, C46.1, C47.1, C48.1, C49.1, C50.1, C51.1, C52.1, C53.1, C54.1, IC1.B7 (VCCO_15_1), IC1.C11 (VCCO_15_2), IC1.C3 (VCCO_34_1), IC1.E6 (VCCO_0_1), IC1.F12 (VCCO_15_3), IC1.G2 (VCCO_34_2), IC1.J14 (VCCO_14_1), IC1.L3 (VCCO_34_3), IC1.M12 (VCCO_14_2), IC1.P5 (VCCO_0_2), IC1.P9 (VCCO_14_3)
- net EECLK: now also U7.2 (SCLK)
- net EECS: now also U7.1 (CS)
- net GND: now also C18.2, C19.2, C20.2, C21.2, C22.2, C23.2, C24.2, C25.2, C26.2, C27.2, C28.2, C29.2, C30.2, C31.2, C32.2, C33.2, C34.2, C35.2, C36.2, C37.2, C38.2, C39.2, C40.2, C41.2, C42.2, C43.2, C44.2, C45.2, C46.2, C47.2, C48.2, C49.2, C50.2, C51.2, C52.2, C53.2, C54.2, C55.2, C56.2, C57.2, C58.2, C59.2, C60.2, C61.2, C62.2, C63.2, C64.2, C65.2, C66.2, C67.2, C68.2, C69.2, C70.2, C71.2, C72.2, C73.2, C74.2, C75.2, FB2.2, IC1.A1 (GND_1), IC1.A15 (GND_2), IC1.B8 (GND_3), IC1.C12 (GND_5), IC1.C2 (GND_4), IC1.D14 (GND_7), IC1.D6 (GND_6), IC1.E4 (GND_8), IC1.E7 (GND_9), IC1.E9 (GND_10), IC1.F10 (GND_12), IC1.F13 (GND_13), IC1.F6 (GND_11), IC1.G3 (GND_14), IC1.G7 (GND_15), IC1.G8 (VREFN_0), IC1.G9 (VP_0), IC1.H10 (GND_17), IC1.H6 (GND_16), IC1.H8 (VN_0), IC1.H9 (VREFP_0), IC1.J13 (GND_19), IC1.J7 (GND_18), IC1.K10 (GND_22), IC1.K6 (GND_20), IC1.K8 (GND_21), IC1.L2 (GND_23), IC1.L7 (GND_24), IC1.L9 (GND_25), IC1.M11 (GND_26), IC1.P13 (GND_29), IC1.P4 (GND_27), IC1.P8 (GND_28), IC1.R1 (GND_30), IC1.R15 (GND_31), J4.10 (SHIELD), J4.6 (VSS), R17.2, SW1.2, SW2.1, SW3.1, U7.5 (GND), U8.4 (GND), X1.1 (GND), X1.40 (GND), X1.41 (GND), X1.42 (GND), X1.43 (GND), X1.44 (GND), X1.45 (GND), X1.46 (GND), X1.47 (GND), X1.48 (GND), X1.49 (GND), Y2.2 (GND)
- net TDO: now also IC1.K4 (TDO_0)
- net TMS: now also IC1.K5 (TMS_0), R16.2; no longer U6.19 (ADBUS3)
- net VCORE: now reaches U6.12 (VCORE)
- net VCORE: now also U6.37 (VCORE), U6.64 (VCORE), C19.1, C20.1, C21.1
- net TCK: now reaches U6.16 (ADBUS0)
- net TCK: now also IC1.E5 (TCK_0), R17.1
- net VCCIO: now reaches U6.20 (VCCIO)
- net VCCIO: now also U6.31 (VCCIO), U6.42 (VCCIO), U6.56 (VCCIO), C22.1, C23.1, C24.1, C25.1
- net VPHY: now reaches U6.4 (VPHY)
- net VPLL: now reaches U6.9 (VPLL)
- net EEDATA: no longer names the net of U6.61 (EEDATA)
- net EEDATA: now also R21.2, U7.4 (DO)
- new net: R21.1, U7.3 (DI)
- new net: IC1.G5 (DONE_0), R22.2
- new net: IC1.J5 (PROGRAM_B_0), R23.1, SW1.1
- new net: IC1.G1 (IO_L12N_T1_MRCC_34), Y2.3 (OUT)
- new net BOOT: R26.1, SW2.2, X1.27 (IO0)
- new net D+: X1.14 (IO20)
- new net D-: X1.13 (IO19)
- new net EN: R25.1, SW3.2, X1.3 (EN)
- new net FLASH_CLK: IC1.F5 (CCLK_0), U8.6 (CLK)
- new net FLASH_CS: U8.1 (~{CS})
- new net FLASH_DI: IC1.H14 (IO_L1P_T0_D00_MOSI_14), U8.2 (DO/IO_{1})
- new net FLASH_DO: IC1.H15 (IO_L1N_T0_D01_DIN_14), U8.5 (DI/IO_{0})
- new net FLASH_HOLD: U8.7 (~{HOLD}/~{RESET}/IO_{3})
- new net FLASH_WP: IC1.J12 (IO_L2P_T0_D02_14), U8.3 (~{WP}/IO_{2})
- new net GNDADC_0: C76.2, FB2.1, IC1.F8 (GNDADC_0)
- new net INT: X1.38 (IO2)
- new net IO11: X1.19 (IO11)
- new net IO12: X1.20 (IO12)
- new net IO13: X1.21 (IO13)
- new net IO14: X1.22 (IO14)
- new net IO4: X1.4 (IO4)
- new net IO5: X1.5 (IO5)
- new net IO6: X1.6 (IO6)
- new net IO7: X1.7 (IO7)
- new net IO8: X1.12 (IO8)
- new net RX: IC1.B5 (IO_L5N_T0_34)
- new net SD_CLK: J4.5 (CLK)
- new net SD_CMD: J4.3 (CMD)
- new net SD_DAT0: J4.7 (DAT0)
- new net SD_DAT3: J4.2 (DAT3/CD)
- new net SD_DET: J4.9 (DET), R24.2
- new net TX: IC1.C5 (IO_L5P_T0_34)
- new net VCCADC_0: C75.1, C76.1, FB1.2, IC1.F9 (VCCADC_0)
- new net VCCBATT_0: IC1.D5 (VCCBATT_0)
- no-connect marks 29 -> 58
Other:
- note added: "BUTTONS"
- note added: "ESP32"
- moved on the sheet: C15, C16, C17, R14, R15, U6, Y1
