File: hardware/processing_board/processing_board.kicad_sch (KiCad schematic)
At the start: 169 parts, among them IC1 XC7S25-2CSGA225I, J1 USB_C_Receptacle_USB2.0_14P, J2 USB_C_Receptacle_USB2.0_14P, J3 S2B-PH-K-S_LF__SN_, J4 Conn_02x07_Counter_Clockwise, SW1 SW_Push, SW2 BOOT_BTN, SW3 RST_BTN, U1 BQ24075RGT, U10 MAX98357A, U11 LP2985-1.8, U2 NCP1117-3.3_SOT223, U3 TPS62821DLC, U4 TPS22917DBV, U6 FT2232HQ, U7 93LCxxA, U8 W25Q32JVSS, U9 W25Q128JVS, X1 ESP32-S3-WROOM-1-N16R8, Y1 Crystal_GND24, Y2 ECS-2520MV-xxx-xx

Commit message: Added 1V0 buck circuit
Parts:
- added C83: 0.1uF, Capacitor_SMD:C_0402_1005Metric, symbol Device:C_Small_US
Connections:
- net +3V3: now also C83.1
- net GND: now also C83.2
Changed lines of the file:
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@@
 	(wire
 		(pts
+			(xy 88.9 168.91) (xy 97.79 168.91)
+		)
+		(stroke
+			(width 0)
+			(type default)
+		)
+	)
+	(wire
+		(pts
 			(xy 57.15 53.34) (xy 57.15 55.88)
 		)
@@
 	(wire
 		(pts
+			(xy 88.9 176.53) (xy 88.9 173.99)
+		)
+		(stroke
+			(width 0)
+			(type default)
+		)
+	)
+	(wire
+		(pts
 			(xy 213.36 391.16) (xy 224.79 391.16)
 		)
@@
 	)
 	(symbol
+		(lib_id "power:GND")
+		(at 88.9 176.53 0)
+		(unit 1)
+		(exclude_from_sim no)
+		(in_bom yes)
+		(on_board yes)
+		(dnp no)
+		(fields_autoplaced yes)
+		(property "Reference" "#PWR0144"
+			(at 88.9 182.88 0)
+			(effects
+				(font
+					(size 1.27 1.27)
+				)
+				(hide yes)
+			)
+		)
+		(property "Value" "GND"
+			(at 88.9 181.61 0)
+			(effects
+				(font
+					(size 1.27 1.27)
+				)
+			)
+		)
+		(property "Footprint" ""
+			(at 88.9 176.53 0)
+			(effects
+				(font
+					(size 1.27 1.27)
+				)
+				(hide yes)
+			)
+		)
+		(property "Datasheet" ""
+			(at 88.9 176.53 0)
+			(effects
+				(font
+					(size 1.27 1.27)
+				)
+				(hide yes)
+			)
+		)
+		(property "Description" "Power symbol creates a global label with name \"GND\" , ground"
+			(at 88.9 176.53 0)
+			(effects
+				(font
+					(size 1.27 1.27)
+				)
+				(hide yes)
+			)
+		)
+		(pin "1"
+		)
+		(instances
+			(project ""
+				(path "/de118238-5cf0-4f20-b51d-7acba9897a1d"
+					(reference "#PWR0144")
+					(unit 1)
+				)
+			)
+		)
+	)
+	(symbol
 		(lib_id "power:+3.3V")
 		(at 236.22 149.86 0)
@@
 					(unit 1)
 				)
+			)
+		)
+	)
+	(symbol
+		(lib_id "Device:C_Small_US")
+		(at 88.9 171.45 0)
+		(unit 1)
+		(exclude_from_sim no)
+		(in_bom yes)
+		(on_board yes)
+		(dnp no)
+		(fields_autoplaced yes)
+		(property "Reference" "C83"
+			(at 91.44 170.3069 0)
+			(effects
+				(font
+					(size 1.27 1.27)
+				)
+				(justify left)
+			)
+		)
+		(property "Value" "0.1uF"
+			(at 91.44 172.8469 0)
+			(effects
+				(font
+					(size 1.27 1.27)
+				)
+				(justify left)
+			)
+		)
+		(property "Footprint" "Capacitor_SMD:C_0402_1005Metric"
+			(at 88.9 171.45 0)
+			(effects
+				(font
+					(size 1.27 1.27)
+				)
+				(hide yes)
+			)
+		)
+		(property "Datasheet" ""
+			(at 88.9 171.45 0)
+			(effects
+				(font
+					(size 1.27 1.27)
+				)
+				(hide yes)
+			)
+		)
+		(property "Description" "capacitor, small US symbol"
+			(at 88.9 171.45 0)
+			(effects
+				(font
+					(size 1.27 1.27)
+				)
+				(hide yes)
+			)
+		)
+		(pin "2"
+		)
+		(pin "1"
+		)
+		(instances
+			(project ""
+				(path "/de118238-5cf0-4f20-b51d-7acba9897a1d"
+					(reference "C83")
+					(unit 1)
+				)
